File: DMH_Multiverter_PCB/DMH_Multiverter_PCB.kicad_sch (KiCad schematic)
At the start: 0 parts

Commit message: Finished schematic
Other:
- sheet Core Circuit ports: added Att A Input, Att A Output, Att B Input, Att B Output; removed none
- sheet Inputs and Outputs ports: added Att A Input Jack, Att A Output Jack, Att B Input Jack, Att B Output Jack; removed none
- sheet Power ports: added none; removed Bus CV, Bus Gate
Changed lines of the file:
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@@
 		(comment 1 "PCB for 5 cm Kosmo format synthesizer module")
 	)
+	(wire
+		(pts
+			(xy 38.1 115.57) (xy 50.8 115.57)
+		)
+		(stroke
+			(width 0)
+			(type default)
+		)
+	)
+	(wire
+		(pts
+			(xy 38.1 111.76) (xy 50.8 111.76)
+		)
+		(stroke
+			(width 0)
+			(type default)
+		)
+	)
+	(wire
+		(pts
+			(xy 38.1 100.33) (xy 50.8 100.33)
+		)
+		(stroke
+			(width 0)
+			(type default)
+		)
+	)
+	(wire
+		(pts
+			(xy 38.1 104.14) (xy 50.8 104.14)
+		)
+		(stroke
+			(width 0)
+			(type default)
+		)
+	)
 	(sheet
-		(at 260.35 16.51)
+		(at 101.6 93.98)
 		(size 20.32 27.94)
 		(fields_autoplaced yes)
@@
 		)
 		(property "Sheetname" "Power"
-			(at 260.35 15.7984 0)
+			(at 101.6 93.2684 0)
 			(effects
 				(font
@@
 		)
 		(property "Sheetfile" "Power.kicad_sch"
-			(at 260.35 45.0346 0)
+			(at 101.6 122.5046 0)
 			(effects
 				(font
@@
 			)
 		)
-		(pin "Bus Gate" output
-			(at 260.35 25.4 180)
-			(effects
-				(font
-					(size 1.27 1.27)
-				)
-				(justify left)
-			)
-		)
-		(pin "Bus CV" output
-			(at 260.35 34.29 180)
-			(effects
-				(font
-					(size 1.27 1.27)
-				)
-				(justify left)
-			)
-		)
 		(instances
-			(project "DMH-Kosmo-5cm-PCB"
+			(project "DMH_Multiverter_PCB"
 				(path "/58f4306d-5387-4983-bb08-41a2313fd315"
 					(page "4")
@@
 	)
 	(sheet
-		(at 120.65 80.01)
-		(size 41.91 38.1)
+		(at 50.8 88.9)
+		(size 38.1 38.1)
 		(fields_autoplaced yes)
 		(stroke
@@
 		)
 		(property "Sheetname" "Core Circuit"
-			(at 120.65 79.2984 0)
+			(at 50.8 88.1884 0)
 			(effects
 				(font
@@
 		)
 		(property "Sheetfile" "Core_Circuit.kicad_sch"
-			(at 120.65 118.6946 0)
+			(at 50.8 127.5846 0)
 			(effects
 				(font
@@
 			)
 		)
+		(pin "Att B Output" output
+			(at 50.8 115.57 180)
+			(effects
+				(font
+					(size 1.27 1.27)
+				)
+				(justify left)
+			)
+		)
+		(pin "Att A Output" output
+			(at 50.8 104.14 180)
+			(effects
+				(font
+					(size 1.27 1.27)
+				)
+				(justify left)
+			)
+		)
+		(pin "Att A Input" input
+			(at 50.8 100.33 180)
+			(effects
+				(font
+					(size 1.27 1.27)
+				)
+				(justify left)
+			)
+		)
+		(pin "Att B Input" input
+			(at 50.8 111.76 180)
+			(effects
+				(font
+					(size 1.27 1.27)
+				)
+				(justify left)
+			)
+		)
 		(instances
-			(project "DMH-Kosmo-5cm-PCB"
+			(project "DMH_Multiverter_PCB"
 				(path "/58f4306d-5387-4983-bb08-41a2313fd315"
 					(page "3")
@@
 	)
 	(sheet
-		(at 17.78 17.78)
-		(size 20.32 118.11)
+		(at 16.51 88.9)
+		(size 21.59 38.1)
 		(fields_autoplaced yes)
 		(stroke
@@
 		)
 		(property "Sheetname" "Inputs and Outputs"
-			(at 17.78 17.0684 0)
+			(at 16.51 88.1884 0)
 			(effects
 				(font
@@
 		)
 		(property "Sheetfile" "Inputs_and_Outputs.kicad_sch"
-			(at 17.78 136.4746 0)
+			(at 16.51 127.5846 0)
 			(effects
 				(font
@@
 			)
 		)
+		(pin "Att A Output Jack" input
+			(at 38.1 104.14 0)
+			(effects
+				(font
+					(size 1.27 1.27)
+				)
+				(justify right)
+			)
+		)
+		(pin "Att B Input Jack" output
+			(at 38.1 111.76 0)
+			(effects
+				(font
+					(size 1.27 1.27)
+				)
+				(justify right)
+			)
+		)
+		(pin "Att A Input Jack" output
+			(at 38.1 100.33 0)
+			(effects
+				(font
+					(size 1.27 1.27)
+				)
+				(justify right)
+			)
+		)
+		(pin "Att B Output Jack" input
+			(at 38.1 115.57 0)
+			(effects
+				(font
+					(size 1.27 1.27)
+				)
+				(justify right)
+			)
+		)
 		(instances
-			(project "DMH-Kosmo-5cm-PCB"
+			(project "DMH_Multiverter_PCB"
 				(path "/58f4306d-5387-4983-bb08-41a2313fd315"
 					(page "2")
