File: DMH_Multiverter_PCB/Power.kicad_sch (KiCad schematic)
At the start: 14 parts, among them J0 Conn_01x01, J100 IDC_02x08, J101 IDC_02x05

Commit message: Finished schematic
Parts:
- removed C3: 47uF, Capacitor_THT:CP_Radial_D4.0mm_P1.50mm, symbol Device:C_Polarized
- removed D1, D3: SB140+, Diode_THT:D_DO-41_SOD81_P10.16mm_Horizontal, symbol SynthStuff:Power_Bus_Schotty_+
- removed D2: SB140-, Diode_THT:D_DO-41_SOD81_P10.16mm_Horizontal, symbol SynthStuff:Power_Bus_Schotty_-
- removed J100: IDC_02x08, SynthStuff:IDC-Header_2x08_P2.54mm_Vertical_Eurorack, symbol SynthStuff:Eurorack_Power_Connector_16Pin
- added C5: 100nF, Capacitor_THT:C_Disc_D4.3mm_W1.9mm_P5.00mm, symbol Device:C
- added U1: TL072, Package_DIP:DIP-8_W7.62mm_Socket, symbol Amplifier_Operational:TL072
- renumbered C4 to C3, C5 to C4, D5 to D1, D4 to D2, J101 to J100
Connections:
- net +5V is gone; now on net GND: C6.1
- net +12V: now also C5.1, U1.8 (V+)
- net -12V: now also C6.2, U1.4 (V-)
- net GND: now also C5.2; no longer C6.2
Other:
- note removed: "Delete what's not needed!"

Commit message: Switched adjustment trimpots position with Rin
... and renumbered the resistors.
Parts:
- J0: now not fitted; now left out of the parts list
Changed lines of the file:
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@@
 		(unit 1)
 		(exclude_from_sim no)
-		(in_bom yes)
+		(in_bom no)
 		(on_board yes)
-		(dnp no)
+		(dnp yes)
 		(property "Reference" "J0"
 			(at 147.32 177.8 90)
