File: DMH_Multiverter_PCB/DMH_Multiverter_PCB.kicad_pcb (KiCad board)
At the start: 2 copper layers, 32 x 75 mm, 24 parts, among them J0 Conn_01x01, J100 IDC_02x05, J200 BackBone_Connector_6pin, J50 Conn_01x06, J60 Conn_01x06, U1 TL072

Commit message: Changed normalled DC offset resistor to 1k
Parts:
- R5: value 10k -> 1k
Changed lines of the file:
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@@
 			)
 		)
-		(property "Value" "10k"
+		(property "Value" "1k"
 			(at 3.81 0 90)
 			(layer "B.SilkS")
