File: DMH_Multiverter_PCB/Inputs_and_Outputs.kicad_sch (KiCad schematic)
At the start: 0 parts

Commit message: Finished schematic
Parts:
- added J1, J10, J11, J12, J13, J14, J15, J16, J17, J18, J19, J2, J20, J21, J22, J3, J4, J5, J6, J7, J8, J9: TS_Jack_6.35mm_Sw, SynthStuff:CUI_MJ-63052A, symbol SynthStuff:TS_Jack_6.35mm_Sw
- added J200: BackBone_Connector_6pin, SynthStuff:IDC-Header_2x03_P2.54mm_Vertical_BackBone, symbol SynthStuff:BackBone_Connector_6pin
- added J50, J60: Conn_01x06, Connector_PinSocket_2.54mm:PinSocket_1x06_P2.54mm_Vertical, symbol Connector_Generic:Conn_01x06
Connections:
- new net: J1.TN, J200.1 (Pin_1), J60.1 (Pin_1)
- new net: J11.T, J12.T, J13.T, J14.TN
- new net: J17.T, J18.T, J19.T, J20.TN
- new net: J200.3 (Pin_3), J3.TN, J60.3 (Pin_3)
- new net: J5.T, J6.T, J7.T, J8.TN
- new net: J20.T, J21.T, J22.T
- new net: J14.T, J15.T, J16.T, J17.TN
- new net: J10.T, J11.TN, J8.T, J9.T
- new net: J2.TN, J200.2 (Pin_2), J60.2 (Pin_2)
- new net: J200.4 (Pin_4), J4.TN, J60.4 (Pin_4)
- new net Att A Input Jack: J1.T, J50.1 (Pin_1)
- new net Att A Output Jack: J2.T, J50.2 (Pin_2)
- new net Att B Input Jack: J3.T, J50.3 (Pin_3)
- new net Att B Output Jack: J4.T, J50.4 (Pin_4)
- new net GND: J1.S, J10.S, J11.S, J12.S, J13.S, J14.S, J15.S, J16.S, J17.S, J18.S, J19.S, J2.S, J20.S, J200.5 (Pin_5), J200.6 (Pin_6), J21.S, J22.S, J3.S, J4.S, J5.S, J50.5 (Pin_5), J50.6 (Pin_6), J6.S, J60.5 (Pin_5), J60.6 (Pin_6), J7.S, J8.S, J9.S
- no-connect marks 0 -> 13

Commit message: Re-routing ongoing
Parts:
- added R7: 100k, Resistor_THT:R_Axial_DIN0207_L6.3mm_D2.5mm_P7.62mm_Horizontal, symbol Device:R_US
- added R8: 82k, Resistor_THT:R_Axial_DIN0207_L6.3mm_D2.5mm_P7.62mm_Horizontal, symbol Device:R_US
Connections:
- net GND: now also J200.3 (Pin_3), R8.1; no longer J200.5 (Pin_5)
- net at J1.TN, J60.1 (Pin_1): now also J3.TN, J60.3 (Pin_3), R7.1, R8.2; no longer J200.1 (Pin_1)
- net at J2.TN, J60.2 (Pin_2): now also J200.1 (Pin_1), J200.4 (Pin_4); no longer J200.2 (Pin_2)
- net at J4.TN, J60.4 (Pin_4): now also J200.2 (Pin_2), J200.5 (Pin_5); no longer J200.4 (Pin_4)
- new net +12V: R7.2

Commit message: Testing out CV offset output feature
Parts:
- R7: value 100k -> 68k
- R8: value 82k -> 100k
Changed lines of the file:
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@@
 			)
 		)
-		(property "Value" "82k"
+		(property "Value" "100k"
 			(at 101.6 237.49 90)
 			(effects
@@
 				)
 				(hide yes)
+			)
+		)
+		(property "Function" ""
+			(at 101.6 241.3 0)
+			(effects
+				(font
+					(size 1.27 1.27)
+				)
 			)
 		)
@@
 			)
 		)
-		(property "Value" "100k"
+		(property "Value" "68k"
 			(at 114.3 237.49 90)
 			(effects

Commit message: Finished Mk2 design
- Changed R7 value to 10k
- Replaced the other resistor with a 5V1 Zener
- Cleaned up schematic
Parts:
- removed R8: 100k, Resistor_THT:R_Axial_DIN0207_L6.3mm_D2.5mm_P7.62mm_Horizontal, symbol Device:R_US
- added D3: ZPD5V1, Diode_THT:D_DO-35_SOD27_P7.62mm_Horizontal, symbol Diode:ZPDxx
- R7: value 68k -> 10k
Connections:
- net GND: now also D3.2 (A)
- net at J1.TN, J3.TN, J60.1 (Pin_1)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: now also D3.1 (K)
Changed lines of the file:
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@@
-	)
-	(symbol
-		(lib_id "Device:R_US")
-		(at 101.6 241.3 90)
-		(unit 1)
-		(exclude_from_sim no)
-		(in_bom yes)
-		(on_board yes)
-		(dnp no)
-		(fields_autoplaced yes)
-		(property "Reference" "R8"
-			(at 101.6 234.95 90)
-			(effects
-				(font
-					(size 1.27 1.27)
-				)
-			)
-		)
-		(property "Value" "100k"
-			(at 101.6 237.49 90)
-			(effects
-				(font
-					(size 1.27 1.27)
-				)
-			)
-		)
-		(property "Footprint" "Resistor_THT:R_Axial_DIN0207_L6.3mm_D2.5mm_P7.62mm_Horizontal"
-			(at 101.854 240.284 90)
-			(effects
-				(font
-					(size 1.27 1.27)
-				)
-				(hide yes)
-			)
-		)
-		(property "Datasheet" "~"
-			(at 101.6 241.3 0)
-			(effects
-				(font
-					(size 1.27 1.27)
-				)
-				(hide yes)
-			)
-		)
-		(property "Description" "Resistor, US symbol"
-			(at 101.6 241.3 0)
-			(effects
-				(font
-					(size 1.27 1.27)
-				)
-				(hide yes)
-			)
-		)
-		(property "Function" ""
-			(at 101.6 241.3 0)
-			(effects
-				(font
-					(size 1.27 1.27)
-				)
-			)
-		)
-		(pin "1"
-		)
-		(pin "2"
-		)
-		(instances
-			(project "DMH_Multiverter_PCB"
-				(path "/58f4306d-5387-4983-bb08-41a2313fd315/ce3fef8b-9f1d-4178-b50b-4a046c030679"
-					(reference "R8")
-					(unit 1)
-				)
-			)
-		)
 	)
 	(symbol
@@
 			)
 		)
-		(property "Value" "68k"
+		(property "Value" "10k"
 			(at 114.3 237.49 90)
 			(effects
@@
 					(unit 1)
 				)
+			)
+		)
+	)
+	(symbol
+		(lib_id "Diode:ZPDxx")
+		(at 101.6 241.3 180)
+		(unit 1)
+		(exclude_from_sim no)
+		(in_bom yes)
+		(on_board yes)
+		(dnp no)
+		(fields_autoplaced yes)
+		(property "Reference" "D3"
+			(at 101.6 234.95 0)
+			(effects
+				(font
+					(size 1.27 1.27)
+				)
+			)
+		)
+		(property "Value" "ZPD5V1"
+			(at 101.6 237.49 0)
+			(effects
+				(font
+					(size 1.27 1.27)
+				)
+			)
+		)
+		(property "Footprint" "Diode_THT:D_DO-35_SOD27_P7.62mm_Horizontal"
+			(at 101.6 236.855 0)
+			(effects
+				(font
+					(size 1.27 1.27)
+				)
+				(hide yes)
+			)
+		)
+		(property "Datasheet" "http://diotec.com/tl_files/diotec/files/pdf/datasheets/zpd1"
+			(at 101.6 241.3 0)
+			(effects
+				(font
+					(size 1.27 1.27)
+				)
+				(hide yes)
+			)
+		)
+		(property "Description" "500mW Zener Diode, DO-35"
+			(at 101.6 241.3 0)
+			(effects
+				(font
+					(size 1.27 1.27)
+				)
+				(hide yes)
+			)
+		)
+		(property "Function" ""
+			(at 101.6 241.3 0)
+			(effects
+				(font
+					(size 1.27 1.27)
+				)
+			)
+		)
+		(pin "1"
+		)
+		(pin "2"
+		)
+		(instances
+			(project ""
+				(path "/58f4306d-5387-4983-bb08-41a2313fd315/ce3fef8b-9f1d-4178-b50b-4a046c030679"
+					(reference "D3")
+					(unit 1)
+				)

Commit message: Switched adjustment trimpots position with Rin
... and renumbered the resistors.
Parts:
- D3: Function (none) -> 5V1
- renumbered R7 to R5
Changed lines of the file:
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@@
 		(dnp no)
 		(fields_autoplaced yes)
-		(property "Reference" "R7"
+		(property "Reference" "R5"
 			(at 114.3 234.95 90)
 			(effects
@@
 			(project "DMH_Multiverter_PCB"
 				(path "/58f4306d-5387-4983-bb08-41a2313fd315/ce3fef8b-9f1d-4178-b50b-4a046c030679"
-					(reference "R7")
+					(reference "R5")
 					(unit 1)
 				)
@@
 		(on_board yes)
 		(dnp no)
-		(fields_autoplaced yes)
 		(property "Reference" "D3"
 			(at 101.6 234.95 0)
@@
 			)
 		)
-		(property "Function" ""
-			(at 101.6 241.3 0)
+		(property "Function" "5V1"
+			(at 101.6 244.856 0)
 			(effects
 				(font
 					(size 1.27 1.27)
+					(thickness 0.254)
+					(bold yes)
+					(italic yes)
 				)
 			)

Commit message: Changed normalled DC offset resistor to 1k
Parts:
- R5: value 10k -> 1k
Changed lines of the file:
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@@
 			)
 		)
-		(property "Value" "10k"
+		(property "Value" "1k"
 			(at 114.3 237.49 90)
 			(effects
