File: DMH_Multiverter_PCB_Conn/DMH_Multiverter_PCB_Conn.kicad_pcb (KiCad board)
At the start: 2 copper layers, 48 x 175 mm, 0 parts

Commit message: Finished conn PCB
Parts:
- added J1: TS_Jack_6.35mm_Sw, SynthStuff:CUI_MJ-63052A, F.Cu at (58.5, 50.0)
- added J10: TS_Jack_6.35mm_Sw, SynthStuff:CUI_MJ-63052A, F.Cu at (91.5, 142.8)
- added J11: TS_Jack_6.35mm_Sw, SynthStuff:CUI_MJ-63052A, F.Cu at (58.5, 159.2)
- added J12: TS_Jack_6.35mm_Sw, SynthStuff:CUI_MJ-63052A, F.Cu at (75.0, 159.2)
- added J13: TS_Jack_6.35mm_Sw, SynthStuff:CUI_MJ-63052A, F.Cu at (91.5, 159.2)
- added J14: TS_Jack_6.35mm_Sw, SynthStuff:CUI_MJ-63052A, F.Cu at (58.5, 175.8)
- added J15: TS_Jack_6.35mm_Sw, SynthStuff:CUI_MJ-63052A, F.Cu at (75.0, 175.8)
- added J16: TS_Jack_6.35mm_Sw, SynthStuff:CUI_MJ-63052A, F.Cu at (91.5, 175.8)
- added J17: TS_Jack_6.35mm_Sw, SynthStuff:CUI_MJ-63052A, F.Cu at (58.5, 192.2)
- added J18: TS_Jack_6.35mm_Sw, SynthStuff:CUI_MJ-63052A, F.Cu at (75.0, 192.2)
- added J19: TS_Jack_6.35mm_Sw, SynthStuff:CUI_MJ-63052A, F.Cu at (91.5, 192.2)
- added J2: TS_Jack_6.35mm_Sw, SynthStuff:CUI_MJ-63052A, F.Cu at (58.5, 67.0)
- added J20: TS_Jack_6.35mm_Sw, SynthStuff:CUI_MJ-63052A, F.Cu at (58.5, 208.8)
- added J21: TS_Jack_6.35mm_Sw, SynthStuff:CUI_MJ-63052A, F.Cu at (75.0, 208.8)
- added J22: TS_Jack_6.35mm_Sw, SynthStuff:CUI_MJ-63052A, F.Cu at (91.5, 208.8)
- added J3: TS_Jack_6.35mm_Sw, SynthStuff:CUI_MJ-63052A, F.Cu at (58.5, 88.2)
- added J4: TS_Jack_6.35mm_Sw, SynthStuff:CUI_MJ-63052A, F.Cu at (58.5, 105.2)
- added J5: TS_Jack_6.35mm_Sw, SynthStuff:CUI_MJ-63052A, F.Cu at (58.5, 126.2)
- added J50: Conn_01x06, Connector_PinHeader_2.54mm:PinHeader_1x06_P2.54mm_Vertical, F.Cu at (69.0, 71.2)
- added J6: TS_Jack_6.35mm_Sw, SynthStuff:CUI_MJ-63052A, F.Cu at (75.0, 126.2)
- added J60: Conn_01x06, Connector_PinHeader_2.54mm:PinHeader_1x06_P2.54mm_Vertical, F.Cu at (89.3, 115.5)
- added J7: TS_Jack_6.35mm_Sw, SynthStuff:CUI_MJ-63052A, F.Cu at (91.5, 126.2)
- added J8: TS_Jack_6.35mm_Sw, SynthStuff:CUI_MJ-63052A, F.Cu at (58.5, 142.8)
- added J9: TS_Jack_6.35mm_Sw, SynthStuff:CUI_MJ-63052A, F.Cu at (75.0, 142.8)
Routing:
- net Net-(J60-Pin_1): track 0.00 -> 108.0 mm
- net Net-(J60-Pin_2): track 0.00 -> 86.6 mm
- net Net-(J17-PadT): track 0.00 -> 54.3 mm
- net Net-(J14-PadT): track 0.00 -> 54.1 mm
- net Net-(J11-PadT): track 0.00 -> 54.1 mm
- net Net-(J10-PadT): track 0.00 -> 54.1 mm
- net Net-(J5-PadT): track 0.00 -> 53.8 mm
- net Net-(J60-Pin_3): track 0.00 -> 39.9 mm
- net Net-(J20-PadT): track 0.00 -> 39.3 mm
- net /Inputs and Outputs/Att B Output Jack: track 0.00 -> 37.1 mm
- net /Inputs and Outputs/Att B Input Jack: track 0.00 -> 25.7 mm
- net Net-(J60-Pin_4): track 0.00 -> 24.2 mm
- net /Inputs and Outputs/Att A Input Jack: track 0.00 -> 21.3 mm
- net /Inputs and Outputs/Att A Output Jack: track 0.00 -> 10.1 mm
- added copper zone on B.Cu, net GND
- added copper zone on F.Cu, net GND
Other:
- outline, holes or cut-outs redrawn

Commit message: Created Gerbers
Other:
- board text added: "Mk1.0 - December 2024"
- board text removed: "Mk1.0 - Month Year"
Changed lines of the file:
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@@
 			(plot_on_all_layers_selection 0x0000000_00000000)
 			(disableapertmacros no)
-			(usegerberextensions no)
+			(usegerberextensions yes)
 			(usegerberattributes yes)
 			(usegerberadvancedattributes yes)
@@
 			(plotinvisibletext no)
 			(sketchpadsonfab no)
-			(subtractmaskfromsilk no)
+			(subtractmaskfromsilk yes)
 			(outputformat 1)
 			(mirror no)
-			(drillshape 1)
+			(drillshape 0)
 			(scaleselection 1)
-			(outputdirectory "")
+			(outputdirectory "Gerbers/")
 		)
 	)
@@
 		)
 		(fp_text user "${REFERENCE}"
-			(at 0 6.35 360)
+			(at 0 6.35 0)
 			(layer "F.Fab")
 			(effects
@@
 		(layer "User.9")
 	)
-	(gr_text "Mk1.0 - Month Year"
+	(gr_text "Mk1.0 - December 2024"
 		(at 74.75 216.5 0)
 		(layer "B.SilkS")
