File: DMH_Multiverter_PCB_Conn/Inputs_and_Outputs.kicad_sch (KiCad schematic)
At the start: 0 parts

Commit message: Finished PCB Conn schematic
Parts:
- added J1, J10, J11, J12, J13, J14, J15, J16, J17, J18, J19, J2, J20, J21, J22, J3, J4, J5, J6, J7, J8, J9: TS_Jack_6.35mm_Sw, SynthStuff:CUI_MJ-63052A, symbol SynthStuff:TS_Jack_6.35mm_Sw
- added J200: BackBone_Connector_6pin, SynthStuff:IDC-Header_2x03_P2.54mm_Vertical_BackBone, symbol SynthStuff:BackBone_Connector_6pin
- added J50, J60: Conn_01x06, Connector_PinHeader_2.54mm:PinHeader_1x06_P2.54mm_Vertical, symbol Connector_Generic:Conn_01x06
Connections:
- new net: J1.TN, J200.1 (Pin_1), J60.1 (Pin_1)
- new net: J2.TN, J200.2 (Pin_2), J60.2 (Pin_2)
- new net: J200.3 (Pin_3), J3.TN, J60.3 (Pin_3)
- new net: J200.4 (Pin_4), J4.TN, J60.4 (Pin_4)
- new net: J11.T, J12.T, J13.T, J14.TN
- new net: J10.T, J11.TN, J8.T, J9.T
- new net: J5.T, J6.T, J7.T, J8.TN
- new net: J17.T, J18.T, J19.T, J20.TN
- new net: J14.T, J15.T, J16.T, J17.TN
- new net: J20.T, J21.T, J22.T
- new net Att A Input Jack: J1.T, J50.1 (Pin_1)
- new net Att A Output Jack: J2.T, J50.2 (Pin_2)
- new net Att B Input Jack: J3.T, J50.3 (Pin_3)
- new net Att B Output Jack: J4.T, J50.4 (Pin_4)
- new net GND: J1.S, J10.S, J11.S, J12.S, J13.S, J14.S, J15.S, J16.S, J17.S, J18.S, J19.S, J2.S, J20.S, J200.5 (Pin_5), J200.6 (Pin_6), J21.S, J22.S, J3.S, J4.S, J5.S, J50.5 (Pin_5), J50.6 (Pin_6), J6.S, J60.5 (Pin_5), J60.6 (Pin_6), J7.S, J8.S, J9.S
- no-connect marks 0 -> 13

Commit message: Finished conn PCB
Parts:
- J1: Function Att A Input -> Att A In
- J10: Function Mult 2 Output 2 -> M 2 Out 2
- J11: Function Mult 3 Input -> Mult 3 In
- J12: Function Mult 3 Output 1 -> M 3 Out 1
- J13: Function Mult 3 Output 2 -> M 3 Out 2
- J14: Function Mult 4 Input -> Mult 4 In
- J15: Function Mult 4 Output 1 -> M 4 Out 1
- J16: Function Mult 4 Output 2 -> M 4 Out 2
- J17: Function Mult 5 Input -> Mult 5 In
- J18: Function Mult 5 Output 1 -> M 5 Out 1
- J19: Function Mult 5 Output 2 -> M 5 Out 2
- J2: Function Att A Output -> Att A Out
- J20: Function Mult 6 Input -> Mult 6 In
- J21: Function Mult 6 Output 1 -> M 6 Out 1
- J22: Function Mult 6 Output 2 -> M 6 Out 2
- J3: Function Att B Input -> Att B In
- J4: Function Att B Output -> Att B Out
- J5: Function Mult 1 Input -> Mult 1 In
- J6: Function Mult 1 Output 1 -> M 1 Out 1
- J7: Function Mult 1 Output 2 -> M 1 Out 2
- J8: Function Mult 2 Input -> Mult 2 In
- J9: Function Mult 2 Output 1 -> M 2 Out 1
Changed lines of the file:
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@@
 			)
 		)
-		(property "Function" "Mult 3 Output 1"
+		(property "Function" "M 3 Out 1"
 			(at 63.5 134.366 0)
 			(effects
@@
 			)
 		)
-		(property "Function" "Mult 2 Output 1"
+		(property "Function" "M 2 Out 1"
 			(at 63.5 83.566 0)
 			(effects
@@
 			)
 		)
-		(property "Function" "Mult 1 Output 1"
+		(property "Function" "M 1 Out 1"
 			(at 63.5 32.766 0)
 			(effects
@@
 			)
 		)
-		(property "Function" "Mult 5 Input"
+		(property "Function" "Mult 5 In"
 			(at 114.3 83.566 0)
 			(effects
@@
 			)
 		)
-		(property "Function" "Att B Output"
+		(property "Function" "Att B Out"
 			(at 25.4 274.066 0)
 			(effects
@@
 			)
 		)
-		(property "Function" "Mult 2 Input"
+		(property "Function" "Mult 2 In"
 			(at 25.4 83.566 0)
 			(effects
@@
 			)
 		)
-		(property "Function" "Mult 1 Output 2"
+		(property "Function" "M 1 Out 2"
 			(at 63.5 58.166 0)
 			(effects
@@
 			)
 		)
-		(property "Function" "Att A Input"
+		(property "Function" "Att A In"
 			(at 25.4 197.866 0)
 			(effects
@@
 			)
 		)
-		(property "Function" "Mult 3 Output 2"
+		(property "Function" "M 3 Out 2"
 			(at 63.5 159.766 0)
 			(effects
@@
 			)
 		)
-		(property "Function" "Mult 2 Output 2"
+		(property "Function" "M 2 Out 2"
 			(at 63.5 108.966 0)
 			(effects
@@
 			)
 		)
-		(property "Function" "Mult 6 Output 2"
+		(property "Function" "M 6 Out 2"
 			(at 152.4 159.766 0)
 			(effects
@@
 			)
 		)
-		(property "Function" "Mult 3 Input"
+		(property "Function" "Mult 3 In"
 			(at 25.4 134.366 0)
 			(effects
@@
 			)
 		)
-		(property "Function" "Att A Output"
+		(property "Function" "Att A Out"
 			(at 25.4 223.266 0)
 			(effects
@@
 			)
 		)
-		(property "Function" "Mult 5 Output 1"
+		(property "Function" "M 5 Out 1"
 			(at 152.4 83.566 0)
 			(effects
@@
 			)
 		)
-		(property "Function" "Mult 4 Output 2"
+		(property "Function" "M 4 Out 2"
 			(at 152.4 58.166 0)
 			(effects
@@
 			)
 		)
-		(property "Function" "Mult 5 Output 2"
+		(property "Function" "M 5 Out 2"
 			(at 152.4 108.966 0)
 			(effects
@@
 			)
 		)
-		(property "Function" "Mult 6 Output 1"
+		(property "Function" "M 6 Out 1"
 			(at 152.4 134.366 0)
 			(effects
@@
 			)
 		)
-		(property "Function" "Mult 1 Input"
+		(property "Function" "Mult 1 In"
 			(at 25.4 32.766 0)
 			(effects
@@
 			)
 		)
-		(property "Function" "Att B Input"
+		(property "Function" "Att B In"
 			(at 25.4 248.666 0)
 			(effects
@@
 			)
 		)
-		(property "Function" "Mult 4 Output 1"
+		(property "Function" "M 4 Out 1"
 			(at 152.4 32.766 0)
 			(effects
@@
 			)
 		)
-		(property "Function" "Mult 4 Input"
+		(property "Function" "Mult 4 In"
 			(at 114.3 32.766 0)
 			(effects
@@
 			)
 		)
-		(property "Function" "Mult 6 Input"
+		(property "Function" "Mult 6 In"
 			(at 114.3 134.366 0)
 			(effects
